File: PCB/LilHelper/LilHelper.kicad_pcb (KiCad board)
At the start: 2 copper layers, 81.8 x 84.1 mm, 27 parts, among them SW1 SW_Push, SW10 SW_Push, SW11 SW_Push, SW12 SW_Push, SW13 RotaryEncoder_Switch, SW2 SW_Push, SW3 SW_Push, SW4 SW_Push, SW5 SW_Push, SW6 SW_Push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

Commit message: Final Commit(Hopefully)
Parts:
- removed D13: 1N4148, Diode_THT:D_DO-35_SOD27_P7.62mm_Horizontal
Connections:
- SW13 pad S1: Net-(U1-GPIO28/ADC2/A2) -> GND
- SW13 pad S2: Net-(D13-A) -> Net-(U1-GPIO28/ADC2/A2)
Routing:
- net Net-(D13-A): track 55.0 -> 0.00 mm, vias 2 -> 0
- net ROW0: track 114.9 -> 95.0 mm
- net GND: track 48.0 -> 63.5 mm
- net Net-(U1-GPIO28/ADC2/A2): track 76.3 -> 74.3 mm
